File: OpenKobold.sch (EAGLE design)
At the start: 7 parts, among them SW1 MSK-12C02_SMD_SPDT_SWITCH, U1 PIC12F675-I/SN

Commit message: Adding part numbers to schematics
Parts:
- BT2: value (none) -> CR1220
- C3: value (none) -> 0.1uF
- R1: value (none) -> 4k
- T1: value (none) -> MMBT2222A
Other:
- moved on the sheet: SG1
Changed lines of the file:
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@@
 <setting verticaltext="up"/>
 </settings>
-<grid distance="0.05" unitdist="inch" unit="inch" style="lines" multiple="1" display="no" altdistance="0.025" altunitdist="inch" altunit="inch"/>
+<grid distance="0.1" unitdist="inch" unit="inch" style="lines" multiple="1" display="no" altdistance="0.01" altunitdist="inch" altunit="inch"/>
 <layers>
 <layer number="1" name="Top" color="4" fill="1" visible="no" active="no"/>
@@
 <part name="GND2" library="supply1" deviceset="GND" device=""/>
 <part name="+3V2" library="supply1" deviceset="+3V3" device=""/>
-<part name="T1" library="transistor" deviceset="*-NPN-" device="SOT23-BEC" technology="MMBT2222ALT1"/>
-<part name="R1" library="rcl" deviceset="R-EU_" device="R0805"/>
+<part name="T1" library="transistor" deviceset="*-NPN-" device="SOT23-BEC" technology="MMBT2222ALT1" value="MMBT2222A"/>
+<part name="R1" library="rcl" deviceset="R-EU_" device="R0805" value="4k"/>
 <part name="GND4" library="supply1" deviceset="GND" device=""/>
 <part name="SG1" library="SparkFun" deviceset="BUZZER" device="PTH"/>
 <part name="+3V3" library="supply1" deviceset="+3V3" device=""/>
-<part name="C3" library="rcl" deviceset="C-EU" device="C0805"/>
+<part name="C3" library="rcl" deviceset="C-EU" device="C0805" value="0.1uF"/>
 <part name="SW1" library="MSK-12C02 SMD Micro Slider Switch SPDT" deviceset="MSK-12C02_SMD_SPDT_SWITCH" device=""/>
 <part name="+3V1" library="supply1" deviceset="+3V3" device=""/>
-<part name="BT2" library="seitan" deviceset="BATTERY" device="-12MM_SMD"/>
+<part name="BT2" library="seitan" deviceset="BATTERY" device="-12MM_SMD" value="CR1220"/>
 </parts>
 <sheets>
@@
 <instance part="R1" gate="G$1" x="88.9" y="58.42"/>
 <instance part="GND4" gate="1" x="104.14" y="63.5"/>
-<instance part="SG1" gate="G$1" x="114.3" y="85.09" rot="MR0"/>
+<instance part="SG1" gate="G$1" x="114.3" y="92.71" rot="MR0"/>
 <instance part="+3V3" gate="G$1" x="116.84" y="68.58" rot="R180"/>
 <instance part="C3" gate="G$1" x="8.89" y="46.99" rot="R180"/>
@@
 <wire x1="116.84" y1="71.12" x2="116.84" y2="78.74" width="0.1524" layer="91"/>
 <pinref part="SG1" gate="G$1" pin="1"/>
-<wire x1="114.3" y1="82.55" x2="114.3" y2="78.74" width="0.1524" layer="91"/>
+<wire x1="114.3" y1="90.17" x2="114.3" y2="78.74" width="0.1524" layer="91"/>
 <wire x1="114.3" y1="78.74" x2="116.84" y2="78.74" width="0.1524" layer="91"/>
 </segment>
@@
 <pinref part="T1" gate="G$1" pin="C"/>
 <pinref part="SG1" gate="G$1" pin="2"/>
-<wire x1="104.14" y1="78.74" x2="104.14" y2="82.55" width="0.1524" layer="91"/>
-<wire x1="104.14" y1="82.55" x2="111.76" y2="82.55" width="0.1524" layer="91"/>
-</segment>
-</net>
+<wire x1="104.14" y1="78.74" x2="104.14" y2="90.17" width="0.1524" layer="91"/>
+<wire x1="104.14" y1="90.17" x2="111.76" y2="90.17" width="0.1524" layer="91"/>
+</segment>
+</net>
